Commit message: updated the xml for leap hand

File: scenes/leap_hand/leap_hand_right.urdf (robot description, URDF)
Before this commit: robot leap_right, 22 links, 21 joints
Links:
- link dip: geometry collision box size=0.014 0.02 0.004; collision box size=0.014 0.02 0.004
- link dip_2: geometry collision box size=0.014 0.02 0.004; collision box size=0.014 0.02 0.004
- link dip_3: geometry collision box size=0.014 0.02 0.004; collision box size=0.014 0.02 0.004
- link fingertip: geometry collision box size=0.014 0.022 0.004; collision box size=0.014 0.022 0.004
- link fingertip_2: geometry collision box size=0.014 0.022 0.004; collision box size=0.014 0.022 0.004
- link fingertip_3: geometry collision box size=0.014 0.022 0.004; collision box size=0.014 0.022 0.004
- link mcp_joint: geometry collision box size=0.014 0.02 0.004; collision box size=0.014 0.02 0.004
- link mcp_joint_2: geometry collision box size=0.014 0.02 0.004; collision box size=0.014 0.02 0.004
- link mcp_joint_3: geometry collision box size=0.014 0.02 0.004; collision box size=0.014 0.02 0.004
- link palm_lower: geometry collision box size=0.004 0.036 0.034; collision box size=0.01 0.12 0.02
- link pip: geometry collision box size=0.034 0.026 0.022; visual mesh filename=meshes/pip.obj
- link pip_2: geometry collision box size=0.034 0.026 0.022; visual mesh filename=meshes/pip.obj
- link pip_3: geometry collision box size=0.034 0.026 0.022; visual mesh filename=meshes/pip.obj
- link thumb_dip: geometry collision box size=0.01 0.024 0.018; collision box size=0.014 0.02 0.004
- link thumb_fingertip: geometry collision box size=0.008 0.024 0.018; collision box size=0.02 0.004 0.03
- link thumb_pip: geometry collision box size=0.014 0.004 0.02; collision box size=0.014 0.004 0.02
- link thumb_temp_base: geometry collision box size=0.034 0.026 0.022; visual mesh filename=meshes/pip.obj

Commit message: added color to the drake cube

File: scenes/leap_hand/leap_hand_right.urdf (robot description, URDF)
Before this commit: robot leap_right, 24 links, 23 joints
Links:
- link obj: geometry collision box size=0.07 0.07 0.07; visual box size=0.0015 0.062 0.062
